File: BreakoutBoard/BreakoutBoard.kicad_pcb (KiCad board)
At the start: 4 copper layers, 112.1 x 130.3 mm, 21 parts, among them J1 QTE-020-01-X-D-A, J10 Conn_01x01_Female, J11 SBH11-NBPC-D12-SM-BK, J2 QTE-020-01-X-D-A, J3 Conn_01x01_Female, J4 Conn_01x01_Female, J5 Conn_01x01_Female, J6 Conn_01x01_Female, J7 Conn_01x01_Female, J8 Conn_01x01_Female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

Commit message: Fixed issues
Connections:
- J10 pad 2: (no net) -> GND
- J3 pad 2: (no net) -> GND
- J4 pad 2: (no net) -> GND
- J5 pad 2: (no net) -> GND
- J6 pad 2: (no net) -> GND
- J7 pad 2: (no net) -> GND
- J8 pad 2: (no net) -> GND
- J9 pad 2: (no net) -> GND
Routing:
- net GND: track 193.7 -> 131.4 mm, vias 0 -> 31

Commit message: Add files via upload
Changed tracks and other minor fixes
Parts:
- moved R2 3.82 mm to (129.7, 91.6)
Routing:
- net /clk0_p: track 163.4 -> 122.1 mm
- net /clk0_n: track 163.2 -> 122.0 mm
- net /tin0_n: track 140.1 -> 115.0 mm
- net /tin0_p: track 140.0 -> 115.1 mm
- net /scl: track 48.7 -> 61.5 mm
- net /sda: track 37.7 -> 45.8 mm
- net LV_RB: track 64.6 -> 71.2 mm
- net GND: track 131.4 -> 136.4 mm
- net /a3: track 2.71 -> 6.52 mm
